File: gpio_breakout.kicad_sch (KiCad schematic)
At the start: 10 parts, among them J10 J_R, J11 J_L, J9 UART, SW3 BTN_USER

Commit message: Created PCB editor, configure for JLCPCB standards
Additionally, created a specific library for castellard jumpers
Parts:
- J10, J11: footprint Connector_PinSocket_2.54mm:PinSocket_1x20_P2.54mm_Vertical -> stm32g431_devboard:PinHeader_1x20_P2.54mm_Vertical
Changed lines of the file:
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@@
 			)
 		)
-		(property "Footprint" "Connector_PinSocket_2.54mm:PinSocket_1x20_P2.54mm_Vertical"
+		(property "Footprint" "stm32g431_devboard:PinHeader_1x20_P2.54mm_Vertical"
 			(at 69.85 107.95 0)
 			(hide yes)
@@
 			)
 		)
-		(property "Footprint" "Connector_PinSocket_2.54mm:PinSocket_1x20_P2.54mm_Vertical"
+		(property "Footprint" "stm32g431_devboard:PinHeader_1x20_P2.54mm_Vertical"
 			(at 189.23 106.68 0)
 			(hide yes)

Commit message: Started PCB placing
Other:
- title: (none) -> ${PROJECT_NAME}, Guillermo Gil
Changed lines of the file:
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@@
 	(generator_version "10.0")
 	(paper "A4")
+	(title_block
+		(title "${PROJECT_NAME}, Guillermo Gil")
+		(rev "v.0.1")
+	)
 	(text "USART2_RX"
 		(exclude_from_sim no)

Commit message: v0.2: low-power redesign — single LDO, ideal diodes, LSE, castellated SWD
Power supply:
- Replace dual LDO (AP2112K + MCP1700) with single TPS7A0233PDBV
  (25 nA Iq nanopower; EN tied to IN per datasheet)
- Replace SS14 Schottky diodes with LM66100 ideal diode controllers
  in diode-OR configuration (CE tied to VOUT for RCB mode)
- Remove jumpers J2 (LDO_SEL), J3 (LED_VBUS), J4 (LED_3V3)
- Replace JST battery connector with castellated header J_VBAT
- Replace J5 IMEAS jumper with 0R bridge
- Rename diode-OR output net to VDC

MCU:
- Add LSE crystal Y1 (32.768 kHz ABS07) with 18 pF load caps
- Dedicate PC14/PC15 to LSE oscillator (removed from J_R breakout)
- Wire BOOT0 net to PB8 (requires nBOOT_SEL=0 option byte)
- Replace VREF_SEL 3-pin jumper with two 0R bridges
- Change reset/boot buttons to C&K PTS810SJM250SMTR (smaller)
- Remove user button SW3

SWD:
- J6 changed from 1x05 THT to 1x06 castellated header
- Pinout follows ST-Link V2 Mini: 3V3/SWCLK/GND/SWDIO/NRST/SWO
- SWO (PB3) shared with GPIO breakout

GPIO breakout:
- Move PA2/PA3 from J_L to J_R (filling former PC14/PC15 slots)
- Add +3V3 and extra GND to J_L in vacated positions
- Break out PC13 to J_R
- J9 UART connector: SMD hand-solderable, no series resistors

Re-annotate all references for sequential numbering.
ERC: clean (with documented exclusion for diode-OR power outputs).
Parts:
- removed C15: 100nF, Capacitor_SMD:C_0603_1608Metric_Pad1.08x0.95mm_HandSolder, symbol Device:C
- removed R10, R9: 1k, Resistor_SMD:R_0603_1608Metric_Pad0.98x0.95mm_HandSolder, symbol Device:R
- removed R8: 10k, Resistor_SMD:R_0603_1608Metric_Pad0.98x0.95mm_HandSolder, symbol Device:R
- removed SW3: BTN_USER, Button_Switch_SMD:SW_SPST_PTS645Sx43SMTR92, symbol Switch:SW_Push
- J5: renamed from J9; footprint Connector_PinHeader_2.54mm:PinHeader_1x04_P2.54mm_Vertical -> Connector_PinHeader_2.54mm:PinHeader_1x04_P2.54mm_Vertical_SMD_Pin1Left
- renumbered D5 to D3, J11 to J3, J10 to J4, R7 to R6
Connections:
- net PC14 is gone; now on net PA3: J4.9 (Pin_9)
- net PC15 is gone; now on net PA2: J4.8 (Pin_8)
- net +3V3: now also J3.19 (Pin_19)
- net GND: now also J3.20 (Pin_20)
- net PA2: now also J5.3 (Pin_3); no longer J3.20 (Pin_20)
- net PA3: now also J5.2 (Pin_2); no longer J3.19 (Pin_19)
- net VBUS renamed VDC
Other:
- moved on the sheet: D3, R6

Commit message: Finish routing
Parts:
- removed J5: UART, Connector_PinHeader_2.54mm:PinHeader_1x04_P2.54mm_Vertical_SMD_Pin1Left, symbol Connector_Generic:Conn_01x04
- J3, J4: footprint stm32g431_devboard:PinHeader_1x20_P2.54mm_Vertical -> Connector_PinHeader_2.54mm:PinHeader_1x20_P2.54mm_Vertical
Connections:
- net +3V3: now also J3.1 (Pin_1), J4.19 (Pin_19); no longer J3.19 (Pin_19), J4.1 (Pin_1)
- net +3V3A: now also J3.19 (Pin_19); no longer J4.20 (Pin_20)
- net GND: now also J4.20 (Pin_20); no longer J3.20 (Pin_20)
- net NRST: now also J3.3 (Pin_3); no longer J4.5 (Pin_5)
- net PA0: now also J3.4 (Pin_4); no longer J4.4 (Pin_4)
- net PA1: now also J3.5 (Pin_5); no longer J4.3 (Pin_3)
- net PA10: now also J4.8 (Pin_8); no longer J3.3 (Pin_3)
- net PA15: now also J4.3 (Pin_3); no longer J4.11 (Pin_11)
- net PA2: now also J3.6 (Pin_6); no longer J4.8 (Pin_8)
- net PA3: now also J3.7 (Pin_7); no longer J4.9 (Pin_9)
- net PA4: now also J3.8 (Pin_8); no longer J3.18 (Pin_18)
- net PA5: now also J3.9 (Pin_9); no longer J3.17 (Pin_17)
- net PA6: now also J3.10 (Pin_10); no longer J3.16 (Pin_16)
- net PA7: now also J3.11 (Pin_11); no longer J3.15 (Pin_15)
- net PA8: now also J4.10 (Pin_10); no longer J3.5 (Pin_5)
- net PA9: now also J4.9 (Pin_9); no longer J3.4 (Pin_4)
- net PB0: now also J3.12 (Pin_12); no longer J3.14 (Pin_14)
- net PB10: now also J3.15 (Pin_15); no longer J3.11 (Pin_11)
- net PB11: now also J3.16 (Pin_16); no longer J3.10 (Pin_10)
- net PB12: now also J3.17 (Pin_17); no longer J3.9 (Pin_9)
- net PB13: now also J3.18 (Pin_18); no longer J3.8 (Pin_8)
- net PB14: now also J4.12 (Pin_12); no longer J3.7 (Pin_7)
- net PB15: now also J4.11 (Pin_11); no longer J3.6 (Pin_6)
- net PB2: now also J3.14 (Pin_14); no longer J3.12 (Pin_12)
- net PB3: now also J4.4 (Pin_4); no longer J4.12 (Pin_12)
- net PB4: now also J4.5 (Pin_5); no longer J4.13 (Pin_13)
- net PB5: now also J4.6 (Pin_6); no longer J4.14 (Pin_14)
- net PB6: now also J4.7 (Pin_7); no longer J4.15 (Pin_15)
- net PB7: now also J4.13 (Pin_13); no longer J4.16 (Pin_16)
- net PB8: now also J4.14 (Pin_14); no longer J4.17 (Pin_17)
- net PB9: now also J4.15 (Pin_15); no longer J4.18 (Pin_18)
- net PC13: now also J4.16 (Pin_16); no longer J4.10 (Pin_10)
- net PF0: now also J4.17 (Pin_17); no longer J4.7 (Pin_7)
- net PF1: now also J4.18 (Pin_18); no longer J4.6 (Pin_6)
- net VDC: now also J4.1 (Pin_1); no longer J3.1 (Pin_1)
- net VREF_EXT_IN: now also J3.20 (Pin_20); no longer J4.19 (Pin_19)
Other:
- note removed: "USART2_RX"
- note removed: "USART2_TX"
