File: mcu.kicad_sch (KiCad schematic)
At the start: 17 parts, among them J6 VREF_SEL, J8 SWD, SW1 BTN_RST, SW2 BOOT

Commit message: Started PCB placing
Other:
- title: (none) -> ${PROJECT_NAME}, Guillermo Gil
Changed lines of the file:
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@@
 	(generator_version "10.0")
 	(paper "A4")
+	(title_block
+		(title "${PROJECT_NAME}, Guillermo Gil")
+		(rev "v.0.1")
+	)
 	(junction
 		(at 148.59 53.34)

Commit message: v0.2: low-power redesign — single LDO, ideal diodes, LSE, castellated SWD
Power supply:
- Replace dual LDO (AP2112K + MCP1700) with single TPS7A0233PDBV
  (25 nA Iq nanopower; EN tied to IN per datasheet)
- Replace SS14 Schottky diodes with LM66100 ideal diode controllers
  in diode-OR configuration (CE tied to VOUT for RCB mode)
- Remove jumpers J2 (LDO_SEL), J3 (LED_VBUS), J4 (LED_3V3)
- Replace JST battery connector with castellated header J_VBAT
- Replace J5 IMEAS jumper with 0R bridge
- Rename diode-OR output net to VDC

MCU:
- Add LSE crystal Y1 (32.768 kHz ABS07) with 18 pF load caps
- Dedicate PC14/PC15 to LSE oscillator (removed from J_R breakout)
- Wire BOOT0 net to PB8 (requires nBOOT_SEL=0 option byte)
- Replace VREF_SEL 3-pin jumper with two 0R bridges
- Change reset/boot buttons to C&K PTS810SJM250SMTR (smaller)
- Remove user button SW3

SWD:
- J6 changed from 1x05 THT to 1x06 castellated header
- Pinout follows ST-Link V2 Mini: 3V3/SWCLK/GND/SWDIO/NRST/SWO
- SWO (PB3) shared with GPIO breakout

GPIO breakout:
- Move PA2/PA3 from J_L to J_R (filling former PC14/PC15 slots)
- Add +3V3 and extra GND to J_L in vacated positions
- Break out PC13 to J_R
- J9 UART connector: SMD hand-solderable, no series resistors

Re-annotate all references for sequential numbering.
ERC: clean (with documented exclusion for diode-OR power outputs).
Parts:
- removed J6: VREF_SEL, Connector_PinHeader_2.54mm:PinHeader_1x03_P2.54mm_Vertical, symbol Connector_Generic:Conn_01x03
- removed J8: SWD, Connector_PinHeader_2.54mm:PinHeader_1x05_P2.54mm_Vertical, symbol Connector_Generic:Conn_01x05
- added C_LSE1, C_LSE2: 18pF, Capacitor_SMD:C_0603_1608Metric_Pad1.08x0.95mm_HandSolder, symbol Device:C
- added J6: Conn_01x06, stm32g431_devboard:PinHeader_1x06_P2.54mm_Vertical_Castellar, symbol Connector_Generic:Conn_01x06
- added R7, R8: 0, Resistor_SMD:R_0603_1608Metric_Pad0.98x0.95mm_HandSolder, symbol Device:R
- added Y1: 32.768 kHz, Crystal:Crystal_SMD_3215-2Pin_3.2x1.5mm, symbol Device:Crystal
- SW1, SW2: footprint Button_Switch_SMD:SW_SPST_TL3342 -> Button_Switch_SMD:SW_SPST_PTS810
- renumbered C11 to C10, C12 to C11, C13 to C12, C14 to C4, C6 to C5, C7 to C6, C8 to C7, C9 to C8, C10 to C9, R5 to R10, R6 to R9
Connections:
- net PB8 is gone; now on net BOOT0: MCU1.45 (PB8)
- net +3V3: now also J6.1 (Pin_1)
- net +3V3A: now also R7.1
- net GND: now also C_LSE1.2, C_LSE2.2, J6.3 (Pin_3)
- net NRST: now also J6.5 (Pin_5)
- net PB3: now also J6.6 (Pin_6)
- net SWCLK: now also J6.2 (Pin_2)
- net SWDIO: now also J6.4 (Pin_4)
- net VREF+: now also R7.2, R8.1
- net VREF_EXT: now also R8.2
- net PC14 renamed OSC32_IN
- net OSC32_IN: now also C_LSE1.1, Y1.1
- net PC15 renamed OSC32_OUT
- net OSC32_OUT: now also C_LSE2.1, Y1.2
Other:
- moved on the sheet: C5, C6, FB1, R10

Commit message: Finish routing
Parts:
- added D5: 1N4148W, Diode_SMD:D_SOD-323, symbol Device:D
- J6: value Conn_01x06 -> Conn_02x06; footprint stm32g431_devboard:PinHeader_1x06_P2.54mm_Vertical_Castellar -> Connector_PinHeader_2.54mm:PinHeader_2x03_P2.54mm_Vertical_SMD
Connections:
- net +3V3: now also D5.1 (K); no longer J6.1 (Pin_1)
- net USB_DM renamed USB_N
- net USB_DP renamed USB_P
- new net: D5.2 (A), J6.1 (Pin_1)
Changed lines of the file:
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@@
 	(wire
 		(pts
-			(xy 257.81 133.35) (xy 260.35 133.35)
-		)
-		(stroke
-			(width 0)
-			(type default)
-		)
-	)
-	(wire
-		(pts
 			(xy 83.82 185.42) (xy 83.82 181.61)
 		)
@@
 	(wire
 		(pts
-			(xy 22.86 26.67) (xy 22.86 36.83)
+			(xy 237.49 127) (xy 237.49 133.35)
 		)
 		(stroke
@@
 	(wire
 		(pts
-			(xy 36.83 26.67) (xy 43.18 26.67)
+			(xy 22.86 26.67) (xy 22.86 36.83)
 		)
 		(stroke
@@
 	(wire
 		(pts
-			(xy 168.91 96.52) (xy 172.72 96.52)
+			(xy 36.83 26.67) (xy 43.18 26.67)
 		)
 		(stroke
@@
 	(wire
 		(pts
-			(xy 62.23 22.86) (xy 62.23 25.4)
+			(xy 168.91 96.52) (xy 172.72 96.52)
 		)
 		(stroke
@@
 	(wire
 		(pts
-			(xy 22.86 36.83) (xy 22.86 39.37)
+			(xy 62.23 22.86) (xy 62.23 25.4)
 		)
 		(stroke
@@
 	(wire
 		(pts
-			(xy 119.38 99.06) (xy 133.35 99.06)
+			(xy 22.86 36.83) (xy 22.86 39.37)
 		)
 		(stroke
@@
 	(wire
 		(pts
-			(xy 119.38 119.38) (xy 133.35 119.38)
+			(xy 119.38 99.06) (xy 133.35 99.06)
 		)
 		(stroke
@@
 	(wire
 		(pts
-			(xy 83.82 185.42) (xy 86.36 185.42)
+			(xy 119.38 119.38) (xy 133.35 119.38)
 		)
 		(stroke
@@
 	(wire
 		(pts
-			(xy 257.81 132.08) (xy 257.81 133.35)
+			(xy 83.82 185.42) (xy 86.36 185.42)
 		)
 		(stroke
@@
 	(wire
 		(pts
+			(xy 250.19 133.35) (xy 260.35 133.35)
+		)
+		(stroke
+			(width 0)
+			(type default)
+		)
+	)
+	(wire
+		(pts
 			(xy 142.24 168.91) (xy 142.24 171.45)
 		)
@@
 	(wire
 		(pts
+			(xy 237.49 133.35) (xy 242.57 133.35)
+		)
+		(stroke
+			(width 0)
+			(type default)
+		)
+	)
+	(wire
+		(pts
 			(xy 259.08 138.43) (xy 259.08 149.86)
 		)
@@
 		)
 	)
-	(hierarchical_label "USB_DM"
+	(hierarchical_label "USB_N"
 		(shape bidirectional)
 		(at 215.9 91.44 0)
@@
 		)
 	)
-	(hierarchical_label "USB_DP"
+	(hierarchical_label "USB_P"
 		(shape bidirectional)
 		(at 215.9 93.98 0)
@@
 	(symbol
 		(lib_id "power:+3V3")
-		(at 257.81 132.08 0)
+		(at 237.49 127 0)
 		(unit 1)
 		(body_style 1)
@@
 		(fields_autoplaced yes)
 		(property "Reference" "#PWR046"
-			(at 257.81 135.89 0)
+			(at 237.49 130.81 0)
 			(hide yes)
 			(show_name no)
@@
 		)
 		(property "Value" "+3V3"
-			(at 257.81 127 0)
+			(at 237.49 121.92 0)
 			(show_name no)
 			(do_not_autoplace no)
@@
 		)
 		(property "Footprint" ""
-			(at 257.81 132.08 0)
+			(at 237.49 127 0)
 			(hide yes)
 			(show_name no)
@@
 		)
 		(property "Datasheet" ""
-			(at 257.81 132.08 0)
+			(at 237.49 127 0)
 			(hide yes)
 			(show_name no)
@@
 		)
 		(property "Description" "Power symbol creates a global label with name \"+3V3\""
-			(at 257.81 132.08 0)
+			(at 237.49 127 0)
 			(hide yes)
 			(show_name no)
@@
 	)
 	(symbol
+		(lib_id "Device:D")
+		(at 246.38 133.35 0)
+		(unit 1)
+		(body_style 1)
+		(exclude_from_sim no)
+		(in_bom yes)
+		(on_board yes)
+		(in_pos_files yes)
+		(dnp no)
+		(fields_autoplaced yes)
+		(property "Reference" "D5"
+			(at 246.38 127 0)
+			(show_name no)
+			(do_not_autoplace no)
+			(effects
+				(font
+					(size 1.27 1.27)
+				)
+			)
+		)
+		(property "Value" "1N4148W"
+			(at 246.38 129.54 0)
+			(show_name no)
+			(do_not_autoplace no)
+			(effects
+				(font
+					(size 1.27 1.27)
+				)
+			)
+		)
+		(property "Footprint" "Diode_SMD:D_SOD-323"
+			(at 246.38 133.35 0)
+			(hide yes)
+			(show_name no)
+			(do_not_autoplace no)
+			(effects
+				(font
+					(size 1.27 1.27)
+				)
+			)
+		)
+		(property "Datasheet" ""
+			(at 246.38 133.35 0)
+			(hide yes)
+			(show_name no)
+			(do_not_autoplace no)
+			(effects
+				(font
+					(size 1.27 1.27)
+				)
+			)
+		)
+		(property "Description" "Diode"
+			(at 246.38 133.35 0)
+			(hide yes)
+			(show_name no)
+			(do_not_autoplace no)
+			(effects
+				(font
+					(size 1.27 1.27)
+				)
+			)
+		)
+		(property "Sim.Device" "D"
+			(at 246.38 133.35 0)
+			(hide yes)
+			(show_name no)
+			(do_not_autoplace no)
+			(effects
+				(font
+					(size 1.27 1.27)
+				)
+			)
+		)
+		(property "Sim.Pins" "1=K 2=A"
+			(at 246.38 133.35 0)
+			(hide yes)
+			(show_name no)
+			(do_not_autoplace no)
+			(effects
+				(font
+					(size 1.27 1.27)
+				)
+			)
+		)
+		(pin "1"
+		)
+		(pin "2"
+		)
+		(instances
+			(project "stm32g431_devboard"
+				(path "/9df7c36b-7f78-4dc7-b3c3-09b2ad159e9d/a5e1f530-8956-4151-8f59-48f85f3d1b34"
+					(reference "D5")
+					(unit 1)
+				)
+			)
+		)
+	)
+	(symbol
 		(lib_id "Device:C")
 		(at 142.24 175.26 0)
@@
 			)
 		)
-		(property "Value" "Conn_01x06"
+		(property "Value" "Conn_02x06"
 			(at 267.97 140.97 0)
 			(show_name no)
@@
 			)
 		)
-		(property "Footprint" "stm32g431_devboard:PinHeader_1x06_P2.54mm_Vertical_Castellar"
+		(property "Footprint" "Connector_PinHeader_2.54mm:PinHeader_2x03_P2.54mm_Vertical_SMD"
 			(at 265.43 138.43 0)
 			(hide yes)
