File: stm32g431_devboard.kicad_pcb (KiCad board)
At the start: 4 copper layers, 60 x 22 mm, 50 parts, among them J1 USB_C_Receptacle_USB2.0_16P, J10 J_R, J11 J_L, J2 LDO_SEL, J3 J_LED_VBUS, J4 J_LED_3V3, J5 J_IMEAS, J6 VREF_SEL, J7 J_EXT_PWR, J8 SWD, J9 UART, SW1 BTN_RST, SW2 BOOT, SW3 BTN_USER, U1 AP2112K-3.3, U2 MCP1700x-330xxTT, U3 USB_ESD

Commit message: Started PCB placing
Parts:
- moved J11 161.4 mm to (57.9, 19.9), turned to -90 degrees
- moved SW3 123.2 mm to (54.0, 11.0), turned to 90 degrees
- moved SW2 120.9 mm to (42.4, 11.2), turned to 90 degrees
- moved MCU1 112.8 mm to (30.0, 11.0), turned to 180 degrees
- moved SW1 101.2 mm to (17.4, 10.8), turned to 90 degrees
- moved J10 98.7 mm to (9.65, 2.11), turned to 90 degrees
- moved J1 71.4 mm to (6.03, 7.70), turned to -90 degrees
- moved J7 64.6 mm to (-30.4, 16.5), turned to 90 degrees

Commit message: Finish routing
Parts:
- removed the C1 at (-35.5, 68.8)
- removed C15: 100nF, Capacitor_SMD:C_0603_1608Metric_Pad1.08x0.95mm_HandSolder
- removed the C4 at (-35.5, 76.3)
- removed the C5 at (-35.5, 78.8)
- removed the D3 at (-22.4, 87.5)
- removed D4: SS14, Diode_SMD:D_SOD-123
- removed the J2 at (-19.4, 69.8)
- removed the J3 at (-23.1, 81.0)
- removed the J4 at (-18.5, 81.0)
- removed J5: J_IMEAS, Connector_PinHeader_2.54mm:PinHeader_1x02_P2.54mm_Vertical
- removed J7: J_EXT_PWR, Connector_JST:JST_PH_S2B-PH-K_1x02_P2.00mm_Horizontal
- removed J8: SWD, Connector_PinHeader_2.54mm:PinHeader_1x05_P2.54mm_Vertical
- removed J9: UART, Connector_PinHeader_2.54mm:PinHeader_1x04_P2.54mm_Vertical
- removed the R10 at (-48.6, 78.8)
- removed the R9 at (-48.6, 76.3)
- removed SW3: BTN_USER, Button_Switch_SMD:SW_SPST_PTS645Sx43SMTR92
- removed the U2 at (-13.9, 74.8)
- added C_LSE1: 18pF, Capacitor_SMD:C_0603_1608Metric_Pad1.08x0.95mm_HandSolder, F.Cu at (37.7, 15.3)
- added C_LSE2: 18pF, Capacitor_SMD:C_0603_1608Metric_Pad1.08x0.95mm_HandSolder, F.Cu at (37.7, 9.73)
- added D5: 1N4148W, Diode_SMD:D_SOD-323, F.Cu at (49.5, 14.2)
- added J1: J_VBAT, Connector_PinHeader_2.54mm:PinHeader_1x02_P2.54mm_Vertical, F.Cu at (2.00, 2.11)
- added R5: 0, Resistor_SMD:R_0603_1608Metric_Pad0.98x0.95mm_HandSolder, F.Cu at (20.6, 14.8)
- added R7: 0, Resistor_SMD:R_0603_1608Metric_Pad0.98x0.95mm_HandSolder, F.Cu at (19.8, 5.00)
- added U3: LM66100DCK, Package_TO_SOT_SMD:SOT-363_SC-70-6, F.Cu at (13.0, 7.47)
- added U4: TPS7A0533PDBV, Package_TO_SOT_SMD:SOT-23-5_HandSoldering, F.Cu at (15.7, 16.2)
- added Y1: 32.768 kHz, Crystal:Crystal_SMD_3215-2Pin_3.2x1.5mm, F.Cu at (37.2, 12.5)
- J2: renamed from J1; footprint Connector_USB:USB_C_Receptacle_GCT_USB4085 -> stm32g431_devboard:USB_C_Receptacle_GCT_USB4085
- J3: renamed from J11; footprint stm32g431_devboard:PinHeader_1x20_P2.54mm_Vertical -> Connector_PinHeader_2.54mm:PinHeader_1x20_P2.54mm_Vertical; moved to B.Cu
- J4: renamed from J10; footprint stm32g431_devboard:PinHeader_1x20_P2.54mm_Vertical -> Connector_PinHeader_2.54mm:PinHeader_1x20_P2.54mm_Vertical; moved to B.Cu
- J6: value VREF_SEL -> Conn_02x06; footprint Connector_PinHeader_2.54mm:PinHeader_1x03_P2.54mm_Vertical -> Connector_PinHeader_2.54mm:PinHeader_2x03_P2.54mm_Vertical_SMD
- R8: value 10k -> 0
- SW1, SW2: footprint Button_Switch_SMD:SW_SPST_TL3342 -> Button_Switch_SMD:SW_SPST_PTS810
- U1: value AP2112K-3.3 -> LM66100DCK; footprint Package_TO_SOT_SMD:SOT-23-5_HandSoldering -> Package_TO_SOT_SMD:SOT-363_SC-70-6
- U2: renamed from U3; footprint Package_TO_SOT_SMD:SOT-23-6_Handsoldering -> Package_TO_SOT_SMD:SOT-23-6
- moved J6 136.0 mm to (53.7, 8.74)
- moved D3 117.2 mm to (42.5, 15.4)
- moved C8 115.8 mm to (36.9, 6.60)
- moved C7 115.1 mm to (36.9, 5.00)
- moved R9 111.7 mm to (52.6, 16.7), turned to -90 degrees
- moved R6 109.9 mm to (46.0, 15.4), turned to 180 degrees
- moved C4 108.3 mm to (44.3, 7.20), turned to 180 degrees
- moved C9 102.6 mm to (26.0, 5.51), turned to 90 degrees
- moved FB1 102.3 mm to (23.2, 5.00), turned to 180 degrees
- moved C6 102.1 mm to (20.1, 7.71), turned to -90 degrees
- moved R10 101.0 mm to (12.8, 5.00), turned to 180 degrees
- moved C5 100.7 mm to (21.7, 7.69), turned to -90 degrees
- moved C11 100.0 mm to (32.1, 17.0), turned to 180 degrees
- moved C12 96.1 mm to (19.9, 17.2), turned to 180 degrees
- moved C10 95.8 mm to (24.5, 15.0), turned to 180 degrees
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- renumbered C16 to C1, C11 to C10, C12 to C11, C13 to C12, C14 to C4, C6 to C5, C7 to C6, C8 to C7, C9 to C8, C10 to C9, D5 to D3, R5 to R10, R7 to R6, R6 to R9
Connections:
- net /MCU/USB_DM renamed /MCU/USB_N
- net /MCU/USB_DP renamed /MCU/USB_P
- net /Power Supply/USB_DM_RAW renamed /Power Supply/USB_RAW_N
- net /Power Supply/USB_DP_RAW renamed /Power Supply/USB_RAW_P
- C1 pad 1: /Power Supply/VBUS_RAW -> VBUS
- C2 pad 1: VBUS -> VDC
- C3 pad 1: Net-(J2-Pin_1) -> Net-(U4-OUT)
- D1 pad 1: Net-(D1-K) -> GND
- D2 pad 1: Net-(D2-K) -> GND
- J2 pad A4: /Power Supply/VBUS_RAW -> VBUS
- J2 pad A9: /Power Supply/VBUS_RAW -> VBUS
- J2 pad B4: /Power Supply/VBUS_RAW -> VBUS
- J2 pad B9: /Power Supply/VBUS_RAW -> VBUS
- J3 pad 1: VBUS -> +3V3
- J3 pad 10: /GPIO Breakout/PB11 -> /GPIO Breakout/PA6
- J3 pad 11: /GPIO Breakout/PB10 -> /GPIO Breakout/PA7
- J3 pad 12: /GPIO Breakout/PB2 -> /GPIO Breakout/PB0
- J3 pad 14: /GPIO Breakout/PB0 -> /GPIO Breakout/PB2
- J3 pad 15: /GPIO Breakout/PA7 -> /GPIO Breakout/PB10
- J3 pad 16: /GPIO Breakout/PA6 -> /GPIO Breakout/PB11
- J3 pad 17: /GPIO Breakout/PA5 -> /GPIO Breakout/PB12
- J3 pad 18: /GPIO Breakout/PA4 -> /GPIO Breakout/PB13
- J3 pad 19: /GPIO Breakout/PA3 -> +3V3A
- J3 pad 20: /GPIO Breakout/PA2 -> /GPIO Breakout/VREF_EXT_IN
- J3 pad 3: /GPIO Breakout/PA10 -> /MCU/NRST
- J3 pad 4: /GPIO Breakout/PA9 -> /GPIO Breakout/PA0
- J3 pad 5: /GPIO Breakout/PA8 -> /GPIO Breakout/PA1
- J3 pad 6: /GPIO Breakout/PB15 -> /GPIO Breakout/PA2
- J3 pad 7: /GPIO Breakout/PB14 -> /GPIO Breakout/PA3
- J3 pad 8: /GPIO Breakout/PB13 -> /GPIO Breakout/PA4
- J3 pad 9: /GPIO Breakout/PB12 -> /GPIO Breakout/PA5
- J4 pad 1: +3V3 -> VDC
- J4 pad 10: /GPIO Breakout/PC13 -> /GPIO Breakout/PA8
- J4 pad 11: /GPIO Breakout/PA15 -> /GPIO Breakout/PB15
- J4 pad 12: /GPIO Breakout/PB3 -> /GPIO Breakout/PB14
- J4 pad 13: /GPIO Breakout/PB4 -> /GPIO Breakout/PB7
- J4 pad 14: /GPIO Breakout/PB5 -> /GPIO Breakout/PB8
- J4 pad 15: /GPIO Breakout/PB6 -> /GPIO Breakout/PB9
- J4 pad 16: /GPIO Breakout/PB7 -> /MCU/PC13
- J4 pad 17: /GPIO Breakout/PB8 -> /GPIO Breakout/PF0
- J4 pad 18: /GPIO Breakout/PB9 -> /GPIO Breakout/PF1
- J4 pad 19: /GPIO Breakout/VREF_EXT_IN -> +3V3
- J4 pad 20: +3V3A -> GND
- J4 pad 3: /GPIO Breakout/PA1 -> /GPIO Breakout/PA15
- J4 pad 4: /GPIO Breakout/PA0 -> /GPIO Breakout/PB3
- J4 pad 5: /MCU/NRST -> /GPIO Breakout/PB4
- J4 pad 6: /GPIO Breakout/PF1 -> /GPIO Breakout/PB5
- J4 pad 7: /GPIO Breakout/PF0 -> /GPIO Breakout/PB6
- J4 pad 8: /GPIO Breakout/PC15 -> /GPIO Breakout/PA10
- J4 pad 9: /GPIO Breakout/PC14 -> /GPIO Breakout/PA9
- J6 pad 1: +3V3A -> Net-(D5-A)
- J6 pad 2: /MCU/VREF+ -> /MCU/SWCLK
- J6 pad 3: /MCU/VREF_EXT -> GND
- MCU1 pad 2: /GPIO Breakout/PC13 -> /MCU/PC13
- MCU1 pad 3: /GPIO Breakout/PC14 -> /MCU/OSC32_IN
- MCU1 pad 4: /GPIO Breakout/PC15 -> /MCU/OSC32_OUT
- R4 pad 2: /Power Supply/+3V3_RAW -> +3V3
- R8 pad 1: +3V3 -> /MCU/VREF+
- R8 pad 2: /GPIO Breakout/PB7 -> /MCU/VREF_EXT
- R9 pad 1: /MCU/BOOT0 -> /GPIO Breakout/PB8
- SW2 pad 2: /MCU/BOOT0 -> /GPIO Breakout/PB8
- U1 pad 1: VBUS -> VBAT_EXT
- U1 pad 3: VBUS -> VDC
- U1 pad 5: Net-(J2-Pin_1) -> unconnected-(U1-ST-Pad5)
- U2 pad 5: /Power Supply/VBUS_RAW -> VBUS
Routing:
- net GND: track 0.00 -> 75.8 mm, vias 0 -> 14
- net /GPIO Breakout/PB3: track 0.00 -> 67.5 mm, vias 0 -> 4
- net /MCU/NRST: track 0.00 -> 40.5 mm, vias 0 -> 2
- net /MCU/SWCLK: track 0.00 -> 39.2 mm, vias 0 -> 2
- net /GPIO Breakout/PB8: track 0.00 -> 37.4 mm, vias 0 -> 2
- net /MCU/SWDIO: track 0.00 -> 34.5 mm, vias 0 -> 2
- net VBUS: track 0.00 -> 31.3 mm, vias 0 -> 4
- net VDC: track 0.00 -> 30.9 mm, vias 0 -> 2
- net /MCU/VREF+: track 0.00 -> 30.8 mm, vias 0 -> 3
- net +3V3: track 0.00 -> 28.3 mm, vias 0 -> 6
- net /GPIO Breakout/PA0: track 0.00 -> 27.5 mm, vias 0 -> 2
- net /GPIO Breakout/PF1: track 0.00 -> 27.0 mm, vias 0 -> 1
- net /Power Supply/USB_RAW_P: track 0.00 -> 25.7 mm, vias 0 -> 3
- net +3V3A: track 0.00 -> 25.1 mm
- net /GPIO Breakout/PB9: track 0.00 -> 24.8 mm, vias 0 -> 2
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- added copper zone on In2.Cu, net +3V3
- added copper zone on In1.Cu, net GND
Other:
- board text added: "+"
- board text added: "-"
- board text added: "BOOT0"
- board text added: "RESET"
- board text added: "SWD"
- board text added: "ULED"
